File: VLC-both/VLC-both.kicad_pcb (KiCad board)
At the start: 2 copper layers, 175.8 x 95.1 mm, 10 parts, among them J1 40HAT, J3 40HAT

Commit message: h
Parts:
- added C1: 100n, Capacitor_SMD:C_0805_2012Metric, F.Cu at (61.6, 23.7)
- added R1: 10k, Resistor_SMD:R_0805_2012Metric, F.Cu at (66.0, 23.7)
- added R2: 10k, Resistor_SMD:R_0805_2012Metric, F.Cu at (61.5, 26.7)
- added R3: 10k, Resistor_SMD:R_0805_2012Metric, F.Cu at (66.0, 26.7)
- added R4: 10k, Resistor_SMD:R_0805_2012Metric, F.Cu at (61.5, 29.6)
- added U1: MCP3008, Package_SO:SOIC-16_3.9x9.9mm_P1.27mm, F.Cu at (55.1, 27.9)
- moved H1 9.44 mm to (217.3, 146.7)
- moved H2 9.44 mm to (159.3, 146.7)
- moved H3 9.44 mm to (217.3, 97.7)
- moved H4 9.44 mm to (159.3, 97.7)
- moved J1 9.44 mm to (212.4, 145.4)
Other:
- board size 175.8 x 95.1 mm -> 185.1 x 96.3 mm

Commit message: c
Parts:
- removed the H1 at (217.3, 146.7)
- removed the H2 at (159.3, 146.7)
- removed the H3 at (217.3, 97.7)
- removed the H4 at (159.3, 97.7)
- added C2: 220u, Capacitor_SMD:C_0805_2012Metric, F.Cu at (91.3, 40.5)
- added C3: 100n-0.1u, Capacitor_SMD:C_0805_2012Metric, F.Cu at (111.6, 44.6)
- added C4: 100n, Capacitor_SMD:C_0805_2012Metric, F.Cu at (103.7, 16.4)
- added C5: 100n, Capacitor_SMD:C_0805_2012Metric, F.Cu at (86.6, 41.3)
- added C6: 100n, Capacitor_SMD:C_0805_2012Metric, F.Cu at (112.1, 13.8)
- added C7: 100n, Capacitor_SMD:C_0805_2012Metric, F.Cu at (117.0, 4.92)
- added J1: light, Connector_PinHeader_2.54mm:PinHeader_1x03_P2.54mm_Vertical, F.Cu at (104.5, 36.6)
- added J2: proxy, Connector_PinHeader_2.54mm:PinHeader_1x03_P2.54mm_Vertical, F.Cu at (99.8, 36.6)
- added J3: dust sense, Connector_PinHeader_2.54mm:PinHeader_1x06_P2.54mm_Vertical, F.Cu at (82.1, 29.9)
- added J4: sound in, Connector_PinHeader_2.54mm:PinHeader_1x04_P2.54mm_Vertical, F.Cu at (86.7, 29.9)
- added J6: Conn_01x03, TerminalBlock:TerminalBlock_Altech_AK300-3_P5.00mm, F.Cu at (77.1, 14.1)
- added Q1: Q_NPN_BEC, Package_TO_SOT_SMD:SOT-23, F.Cu at (119.5, 36.7)
- added R10: 100, Resistor_SMD:R_0805_2012Metric, F.Cu at (121.4, 7.84)
- added R11: 10k, Resistor_SMD:R_0805_2012Metric, F.Cu at (121.4, 10.8)
- added R12: 10k, Resistor_SMD:R_0805_2012Metric, F.Cu at (121.4, 4.89)
- added R13: 10k, Resistor_SMD:R_0805_2012Metric, F.Cu at (116.5, 13.8)
- added R14: 10k, Resistor_SMD:R_0805_2012Metric, F.Cu at (117.0, 7.90)
- added R5: 10k, Resistor_SMD:R_0805_2012Metric, F.Cu at (91.0, 43.5)
- added R6: 90k, Resistor_SMD:R_0805_2012Metric, F.Cu at (126.9, 27.3)
- added R7: 10k, Resistor_SMD:R_0805_2012Metric, F.Cu at (119.5, 31.5)
- added R8: DNP, Resistor_SMD:R_0805_2012Metric, F.Cu at (126.9, 30.3)
- added R9: 10k, Resistor_SMD:R_0805_2012Metric, F.Cu at (113.4, 35.8)
- added U2: LM4040DBZ-4.1, Package_TO_SOT_SMD:SOT-23, F.Cu at (112.3, 10.1)
- added U3: MCP3008, Package_SO:SOIC-16_3.9x9.9mm_P1.27mm, F.Cu at (93.3, 33.3)
- added U4: CN240A05, Package_SIP:SIP4_Sharp-SSR_P7.62mm_Straight, F.Cu at (82.3, 22.8)
- added U5: LM4040DBZ-4.1, Package_TO_SOT_SMD:SOT-23, F.Cu at (112.3, 5.64)
- added U6: MCP3008, Package_SO:SOIC-16_3.9x9.9mm_P1.27mm, F.Cu at (105.7, 9.14)
- C1: value 100n -> 100n-0.1u
- R1: value 10k -> 150
- R3: value 10k -> 100
- U1: value MCP3008 -> LM35-LP; footprint Package_SO:SOIC-16_3.9x9.9mm_P1.27mm -> Connector_PinHeader_2.54mm:PinHeader_1x03_P2.54mm_Vertical
- moved U1 64.8 mm to (119.7, 22.6)
- moved R2 59.3 mm to (119.3, 40.4)
- moved R3 53.4 mm to (117.0, 10.9)
- moved R4 48.3 mm to (109.0, 38.7)
- moved R1 44.7 mm to (109.0, 35.8)
- moved C1 32.4 mm to (86.6, 44.3)
- renumbered J1 to J5, J3 to J7
Connections:
- C1 pad 1: +5V -> +3V3
- J5 pad 19: unconnected-(J1-Pad19) -> MOSI2
- J5 pad 21: unconnected-(J1-Pad21) -> MISO2
- J5 pad 23: unconnected-(J1-Pad23) -> CLK2
- J5 pad 24: unconnected-(J1-Pad24) -> SS2
- J7 pad 19: unconnected-(J3-Pad19) -> MOSI1
- J7 pad 21: unconnected-(J3-Pad21) -> MISO1
- J7 pad 23: unconnected-(J3-Pad23) -> CLK1
- J7 pad 24: unconnected-(J3-Pad24) -> SS1
- R1 pad 1: +3V3 -> +5V
- R1 pad 2: CLK1 -> Net-(J3-Pad1)
- R2 pad 1: +3V3 -> +5V
- R2 pad 2: MISO1 -> /ADC3
- R3 pad 1: +3V3 -> /Vref1
- R3 pad 2: MOSI1 -> +5V
- R4 pad 2: SS1 -> CLK2
- U1 pad 1: unconnected-(U1-Pad1) -> +5V
- U1 pad 2: unconnected-(U1-Pad2) -> /ADC0
- U1 pad 3: unconnected-(U1-Pad3) -> GND

Commit message: r
Parts:
- added C8: 100n, Capacitor_SMD:C_0805_2012Metric, F.Cu at (229.9, 57.5)
- added C9: 100n, Capacitor_SMD:C_0805_2012Metric, F.Cu at (220.6, 61.5)
- added H4: 3mm_Mounting_Hole, project_footprints:NPTH_3mm_ID, F.Cu at (72.3, 148.8)
- added H4: 3mm_Mounting_Hole, project_footprints:NPTH_3mm_ID, F.Cu at (130.3, 148.8)
- added J8: sound in, Connector_PinHeader_2.54mm:PinHeader_1x04_P2.54mm_Vertical, F.Cu at (220.7, 50.1)
- added R15: DNP, Resistor_SMD:R_0805_2012Metric, F.Cu at (234.3, 57.5)
- added R16: DNP, Resistor_SMD:R_0805_2012Metric, F.Cu at (241.7, 52.2)
- added R17: 10k, Resistor_SMD:R_0805_2012Metric, F.Cu at (229.8, 60.5)
- added R18: 20k, Resistor_SMD:R_0805_2012Metric, F.Cu at (234.3, 60.4)
- added R19: 10k, Resistor_SMD:R_0805_2012Metric, F.Cu at (241.7, 49.2)
- added RV1: R_Potentiometer, Potentiometer_THT:Potentiometer_Piher_PT-6-V_Vertical, F.Cu at (232.9, 54.4)
- added RV2: R_Potentiometer, Potentiometer_THT:Potentiometer_Piher_PT-6-V_Vertical, F.Cu at (224.6, 54.4)
- added TH1: Thermistor, Connector_PinHeader_2.54mm:PinHeader_1x02_P2.54mm_Vertical, F.Cu at (225.3, 58.3)
- moved J6 171.7 mm to (220.4, 108.8)
- moved U4 171.7 mm to (225.5, 117.5)
- moved C2 89.9 mm to (174.0, 75.7)
- moved R2 89.9 mm to (202.0, 75.6)
- moved R3 89.9 mm to (199.8, 46.0)
- moved R5 89.9 mm to (173.8, 78.7)
- moved U6 89.9 mm to (188.4, 44.3)
- moved C1 89.9 mm to (169.4, 79.5)
- moved C3 89.9 mm to (194.4, 79.8)
- moved C4 89.9 mm to (186.4, 51.5)
- moved C5 89.9 mm to (169.4, 76.5)
- moved C6 89.9 mm to (194.9, 49.0)
- moved Q1 89.9 mm to (202.3, 71.9)
- moved R10 89.9 mm to (204.2, 43.0)
- moved R11 89.9 mm to (204.2, 46.0)
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Connections:
- C2 pad 1: +5V -> Net-(J3-Pad1)
- J5 pad 36: unconnected-(J5-Pad36) -> /proxy_out
- J5 pad 38: unconnected-(J5-Pad38) -> /audio_digital_out
- J5 pad 40: unconnected-(J5-Pad40) -> /V-O
- J7 pad 38: unconnected-(J7-Pad38) -> /Comparator1
- J7 pad 40: unconnected-(J7-Pad40) -> /Comparator2
- U6 pad 2: /ADC1 -> unconnected-(U6-Pad2)
- U6 pad 3: /ADC2 -> unconnected-(U6-Pad3)
- U6 pad 4: /ADC3 -> unconnected-(U6-Pad4)
- U6 pad 5: /ADC4 -> unconnected-(U6-Pad5)
- U6 pad 6: /ADC5 -> unconnected-(U6-Pad6)
- U6 pad 7: /ADC6 -> unconnected-(U6-Pad7)
- U6 pad 8: /ADC7 -> unconnected-(U6-Pad8)
Other:
- board size 185.1 x 96.3 mm -> 98.1 x 98.3 mm

Commit message: t
Parts:
- removed the H4 at (72.3, 148.8)
- removed the H4 at (130.3, 148.8)
- removed the J8 at (220.7, 50.1)
- added IC1: TC75S59FU_TE85L,F_, SamacSys_Parts:TC75S59FUTE85LF, F.Cu at (43.3, 122.1)
- added IC2: TC75S59FU_TE85L,F_, SamacSys_Parts:TC75S59FUTE85LF, F.Cu at (52.2, 142.8)
- added J7: Analof light in, Connector_PinHeader_2.54mm:PinHeader_1x06_P2.54mm_Vertical, F.Cu at (38.2, 130.3)
- added R15: de calculat, Resistor_SMD:R_0805_2012Metric, F.Cu at (42.3, 125.7)
- added R16: de calculat, Resistor_SMD:R_0805_2012Metric, F.Cu at (46.1, 125.8)
- added U7: ADS7041xDCU, Package_SO:VSSOP-8_2.3x2mm_P0.5mm, F.Cu at (44.3, 110.5)
- C1: renamed from C2; footprint Capacitor_SMD:C_0805_2012Metric -> Capacitor_SMD:CP_Elec_6.3x7.7
- moved R11 208.0 mm to (44.5, 118.4), turned to 180 degrees
- moved R14 207.7 mm to (44.4, 114.0), turned to 180 degrees
- moved RV1 207.4 mm to (42.7, 137.1), turned to -90 degrees
- moved R13 197.9 mm to (44.4, 116.2)
- moved R10 196.0 mm to (48.0, 118.4), turned to 180 degrees
- moved C7 193.1 mm to (47.6, 121.2), turned to 180 degrees
- moved R12 190.2 mm to (48.0, 116.2)
- moved RV2 186.5 mm to (55.6, 133.3), turned to 180 degrees
- moved C8 182.6 mm to (56.5, 141.9), turned to 180 degrees
- moved R21 171.0 mm to (61.6, 143.7)
- moved R18 170.8 mm to (62.7, 141.6)
- moved R19 170.2 mm to (67.6, 141.7), turned to 180 degrees
- moved R17 164.6 mm to (63.4, 128.4), turned to 90 degrees
- moved R20 161.5 mm to (68.7, 143.8), turned to 180 degrees
- moved C9 160.5 mm to (63.4, 124.8), turned to 90 degrees
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- renumbered C3 to C2, C4 to C3, C5 to C4, C1 to C5, C8 to C7, C9 to C8, C7 to C9, J3 to J1, J4 to J2, J5 to J3, J6 to J4, J1 to J5, J2 to J6, J7 to J8, R6 to R1, R15 to R10, R16 to R11, R17 to R12, R18 to R13, R19 to R14, R10 to R17, R11 to R18, R12 to R19, R8 to R2, R13 to R20, R14 to R21, R1 to R3, R3 to R4, R2 to R5, R4 to R6, R5 to R7, R7 to R8, U4 to U2, U2 to U3, U3 to U4
Connections:
- net Net-(J6-Pad2) renamed /L1
- C3 pad 1: /Vref1 -> /Vref2
- J4 pad 1: unconnected-(J6-Pad1) -> /L2
- J4 pad 3: Net-(J6-Pad3) -> unconnected-(J4-Pad3)
- R4 pad 1: /Vref1 -> /Vref2
- RV1 pad 1: /Vref1 -> IN2
- RV2 pad 1: IN2 -> /Vref1
- U2 pad 2: Net-(J6-Pad3) -> /L2
- U3 pad 1: /Vref1 -> /Vref2
- U4 pad 15: /Vref1 -> /Vref2
- U6 pad 1: /ADC0 -> /ADC0_1
Routing:
- added copper zone on B.Cu, net GND
Other:
- board size 98.1 x 98.3 mm -> 98.4 x 97.7 mm
- board text added: "RECEIVER"
- board text added: "TRANSMITTER"
