File: VLC-both/VLC-both.kicad_pcb (KiCad board)
At the start: 2 copper layers, 98.4 x 97.7 mm, 58 parts, among them IC1 TC75S59FU_TE85L,F_, IC2 TC75S59FU_TE85L,F_, J1 dust sense, J2 sound in, J3 40HAT, J4 Conn_01x03, J5 light, J6 proxy, J7 Analof light in, J8 40HAT, Q1 Q_NPN_BEC, U1 LM35-LP, U2 CN240A05, U3 LM4040DBZ-4.1, U4 MCP3008, U5 LM4040DBZ-4.1, U6 MCP3008, U7 ADS7041xDCU

Commit message: r
Parts:
- added C10: 1u, Capacitor_SMD:C_0805_2012Metric, F.Cu at (49.9, 107.7)
- added C11: 1u, Capacitor_SMD:C_0805_2012Metric, F.Cu at (54.3, 113.0)
- added C12: 1u, Capacitor_SMD:C_0805_2012Metric, F.Cu at (46.7, 108.5)
- added FID1: Fiducial, Fiducial:Fiducial_0.5mm_Mask1mm, F.Cu at (84.1, 65.9)
- added FID2: Fiducial, Symbol:WEEE-Logo_4.2x6mm_SilkScreen, F.Cu at (71.8, 137.3)
- added FID3: Fiducial, Fiducial:Fiducial_0.5mm_Mask1mm, F.Cu at (98.1, 143.9)
- added FID4: Fiducial, Symbol:WEEE-Logo_4.2x6mm_SilkScreen, F.Cu at (87.2, 110.6)
- added R22: DNP, Resistor_SMD:R_0805_2012Metric, F.Cu at (46.7, 112.1)
- added R23: 100, Resistor_SMD:R_0805_2012Metric, F.Cu at (55.6, 103.8)
- added R24: 10k, Resistor_SMD:R_0805_2012Metric, F.Cu at (52.5, 143.8)
- added R25: 10k, Resistor_SMD:R_0805_2012Metric, F.Cu at (48.9, 143.8)
- added R26: 10k, Resistor_SMD:R_0805_2012Metric, F.Cu at (50.0, 141.7)
- added U8: LM4040DBZ-3, Package_TO_SOT_SMD:SOT-23, F.Cu at (52.0, 104.7)
- added kibuzzard-62B56940: G***, kibuzzard-62B56940, F.Cu at (112.4, 102.0)
- added kibuzzard-62B56940: G***, kibuzzard-62B56940, F.Cu at (87.9, 134.4)
- added kibuzzard-62B56AED: G***, kibuzzard-62B56AED, F.Cu at (115.1, 58.4)
- added kibuzzard-62B56B9A: G***, kibuzzard-62B56B9A, F.Cu at (112.3, 106.7)
- added kibuzzard-62B56B9A: G***, kibuzzard-62B56B9A, F.Cu at (87.8, 139.1)
- added kibuzzard-62B56CEF: G***, kibuzzard-62B56CEF, F.Cu at (84.4, 88.6)
- added kibuzzard-62B56CEF: G***, kibuzzard-62B56CEF, F.Cu at (93.1, 113.5)
- added kibuzzard-62B56CEF: G***, kibuzzard-62B56CEF, F.Cu at (84.4, 104.4)
- added kibuzzard-62B56CEF: G***, kibuzzard-62B56CEF, F.Cu at (104.1, 113.5)
- added kibuzzard-62B56DD8: G***, kibuzzard-62B56DD8, F.Cu at (85.4, 77.2)
- added kibuzzard-62B56DD8: G***, kibuzzard-62B56DD8, F.Cu at (85.0, 93.5)
- added kibuzzard-62B56DD8: G***, kibuzzard-62B56DD8, F.Cu at (109.4, 112.8)
- added kibuzzard-62B56DD8: G***, kibuzzard-62B56DD8, F.Cu at (122.8, 112.8)
- added kibuzzard-62B56DD8: G***, kibuzzard-62B56DD8, F.Cu at (98.4, 112.8)
- added kibuzzard-62B56E37: G***, kibuzzard-62B56E37, F.Cu at (87.1, 74.7)
- added kibuzzard-62B56E37: G***, kibuzzard-62B56E37, F.Cu at (95.8, 111.1)
- added kibuzzard-62B56E37: G***, kibuzzard-62B56E37, F.Cu at (86.7, 91.1)
- added kibuzzard-62B57016: G***, kibuzzard-62B57016, F.Cu at (106.9, 111.8)
- added kibuzzard-62B57037: G***, kibuzzard-62B57037, F.Cu at (114.9, 112.2)
- added kibuzzard-62B57048: G***, kibuzzard-62B57048, F.Cu at (118.4, 112.9)
- added kibuzzard-62B57048: G***, kibuzzard-62B57048, F.Cu at (85.3, 79.8)
- added kibuzzard-62B57119: G***, kibuzzard-62B57119, F.Cu at (81.3, 108.3)
- added kibuzzard-62B5717A: G***, kibuzzard-62B5717A, F.Cu at (80.7, 67.2)
- added kibuzzard-62B5718E: G***, kibuzzard-62B5718E, F.Cu at (86.9, 82.5)
- added kibuzzard-62B571D5: G***, kibuzzard-62B571D5, F.Cu at (84.7, 96.1)
- added kibuzzard-62B57254: G***, kibuzzard-62B57254, F.Cu at (85.0, 98.7)
- moved RV2 10.9 mm to (66.2, 130.8)
- moved C8 10.5 mm to (46.1, 143.1), turned to -90 degrees
- moved IC2 9.27 mm to (42.9, 143.1), turned to 180 degrees
- moved U5 8.06 mm to (72.4, 131.8)
- moved C9 8.06 mm to (71.5, 124.6)
- moved R17 8.06 mm to (71.5, 128.2)
- moved U6 8.06 mm to (64.8, 125.0)
- moved C6 7.88 mm to (69.2, 131.8)
- moved IC1 6.58 mm to (49.8, 121.7)
- moved J7 6.58 mm to (44.7, 129.9)
- moved R10 6.58 mm to (54.6, 118.0)
- moved R16 6.58 mm to (52.7, 125.4)
- moved U7 6.58 mm to (50.8, 110.1)
- moved C7 6.58 mm to (54.2, 120.8)
- moved R11 6.58 mm to (51.0, 118.0)
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Connections:
- net Net-(IC1-Pad1) renamed /IN-2
- net Net-(IC1-Pad3) renamed /IN+2
- net Net-(IC2-Pad1) renamed /IN-1
- net Net-(IC2-Pad3) renamed /IN+1
- C7 pad 2: +3V3 -> +3.3VA
- C8 pad 2: +3V3 -> +3.3VA
- C9 pad 1: +5V -> +5VA
- IC1 pad 5: +3V3 -> +3.3VA
- IC2 pad 5: +3V3 -> +3.3VA
- J3 pad 15: unconnected-(J3-Pad15) -> /audio_digital_out
- J3 pad 35: unconnected-(J3-Pad35) -> /V-O
- J3 pad 36: /proxy_out -> unconnected-(J3-Pad36)
- J3 pad 37: unconnected-(J3-Pad37) -> /proxy_out
- J3 pad 38: /audio_digital_out -> unconnected-(J3-Pad38)
- J3 pad 40: /V-O -> /light
- J8 pad 1: +3V3 -> +3.3VA
- J8 pad 17: +3V3 -> +3.3VA
- J8 pad 2: +5V -> +5VA
- J8 pad 35: unconnected-(J8-Pad35) -> MISO3
- J8 pad 36: unconnected-(J8-Pad36) -> SS3
- J8 pad 37: unconnected-(J8-Pad37) -> /Comparator1
- J8 pad 38: /Comparator1 -> unconnected-(J8-Pad38)
- J8 pad 4: +5V -> +5VA
- J8 pad 40: /Comparator2 -> CLK3
- R17 pad 2: +5V -> +5VA
- R18 pad 1: +3V3 -> +3.3VA
- R19 pad 1: +3V3 -> +3.3VA
- R20 pad 1: +3V3 -> +3.3VA
- R21 pad 1: +3V3 -> +3.3VA
- U6 pad 16: +5V -> +5VA
- U7 pad 1: unconnected-(U7-Pad1) -> +3.3VA
- U7 pad 2: unconnected-(U7-Pad2) -> CLK3
- U7 pad 3: unconnected-(U7-Pad3) -> MISO3
- U7 pad 4: unconnected-(U7-Pad4) -> SS3
- U7 pad 6: /ADC1_1 -> /input
- U7 pad 7: unconnected-(U7-Pad7) -> /ref3
Routing:
- net +3.3VA: track 0.00 -> 120.2 mm, vias 0 -> 11
- net /audio_digital_out: track 0.00 -> 50.0 mm, vias 0 -> 5
- net CLK3: track 0.00 -> 49.6 mm, vias 0 -> 2
- net SS3: track 0.00 -> 49.4 mm, vias 0 -> 2
- net +5VA: track 0.00 -> 48.0 mm, vias 0 -> 2
- net MISO3: track 0.00 -> 46.0 mm, vias 0 -> 2
- net +3V3: track 71.3 -> 116.4 mm, vias 5 -> 9
- net /Vref1: track 0.00 -> 43.9 mm, vias 0 -> 2
- net /ADC0_1: track 0.00 -> 28.1 mm, vias 0 -> 4
- net /proxy_out: track 0.00 -> 27.7 mm
- net MOSI1: track 0.00 -> 26.2 mm, vias 0 -> 4
- net SS1: track 0.00 -> 24.2 mm
- net GND: track 31.9 -> 55.6 mm, vias 20 -> 37
- net MISO1: track 0.00 -> 22.6 mm, vias 0 -> 2
- net /IN-1: track 0.00 -> 22.1 mm
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- added copper zone on F.Cu, net +5V
- added copper zone on F.Cu, net +5VA
Other:
- outline, holes or cut-outs redrawn
- board text removed: "RECEIVER"
- board text removed: "TRANSMITTER"

Commit message: r
Parts:
- added ?: , , F.Cu at (76.5, 106.2)
- added kibuzzard-62B58D0E: G***, kibuzzard-62B58D0E, F.Cu at (86.7, 126.2)
- added kibuzzard-62B59380: G***, kibuzzard-62B59380, F.Cu at (39.6, 122.2)
- added kibuzzard-62B59390: G***, kibuzzard-62B59390, F.Cu at (39.5, 127.5)
- added kibuzzard-62B59408: G***, kibuzzard-62B59408, F.Cu at (39.9, 119.8)
- added kibuzzard-62B59413: G***, kibuzzard-62B59413, F.Cu at (39.9, 124.8)
- added kibuzzard-62B5942E: G***, kibuzzard-62B5942E, F.Cu at (40.6, 130.0)
- added kibuzzard-62B594DE: G***, kibuzzard-62B594DE, F.Cu at (50.2, 136.8)
- added kibuzzard-62B594FE: G***, kibuzzard-62B594FE, F.Cu at (54.4, 131.8)
- moved FID2 42.3 mm to (39.6, 109.7)
Routing:
- net /ref3: track 10.3 -> 37.2 mm
- net +3.3VA: track 120.2 -> 141.0 mm

Commit message: f
Parts:
- removed ?: , 
- removed the H4 at (130.3, 58.3)
- removed the H4 at (130.4, 116.3)
- removed the H4 at (81.5, 116.3)
- added H4: 3mm_Mounting_Hole, project_footprints:NPTH_3mm_ID, F.Cu at (130.4, 58.3)
- added H4: 3mm_Mounting_Hole, project_footprints:NPTH_3mm_ID, F.Cu at (130.4, 116.4)
- added H4: 3mm_Mounting_Hole, project_footprints:NPTH_3mm_ID, F.Cu at (81.5, 116.4)
- added J9: Conn_01x01, Connector_PinHeader_2.54mm:PinHeader_1x01_P2.54mm_Vertical, F.Cu at (76.4, 106.5)
- added R27: 10k, Resistor_SMD:R_0805_2012Metric, F.Cu at (122.7, 72.6)
- added R28: 10k, Resistor_SMD:R_0805_2012Metric, F.Cu at (82.3, 143.5)
- added SW1: SW_SPST, SamacSys_Parts:PTS526SM15SMTR2LFS, F.Cu at (119.6, 78.3)
- added SW2: SW_SPST, SamacSys_Parts:PTS526SM15SMTR2LFS, F.Cu at (76.5, 141.7)
- added kibuzzard-62B5CDB9: G***, kibuzzard-62B5CDB9, F.Cu at (85.2, 139.9)
- added kibuzzard-62B5CDB9: G***, kibuzzard-62B5CDB9, F.Cu at (119.6, 87.0)
- moved kibuzzard-62B56940 2.78 mm to (88.1, 131.6)
- moved kibuzzard-62B56B9A 2.78 mm to (88.0, 136.3)
- moved kibuzzard-62B58D0E 0.72 mm to (86.6, 125.5)
- renumbered IC2 to IC1, IC1 to IC2
Connections:
- J3 pad 11: unconnected-(J3-Pad11) -> /reset1
- J8 pad 11: unconnected-(J8-Pad11) -> /reset2
Routing:
- net /reset1: track 0.00 -> 17.2 mm, vias 0 -> 2
- net /reset2: track 0.00 -> 12.7 mm, vias 0 -> 1
- net GND: track 55.6 -> 60.1 mm, vias 37 -> 41
- net +5VA: track 48.0 -> 44.4 mm
- net +3V3: track 116.4 -> 118.3 mm
- net +3.3VA: track 141.0 -> 142.0 mm
- net /ref3: track 37.2 -> 36.6 mm

Commit message: r
Parts:
- removed J9: Conn_01x01, Connector_PinHeader_2.54mm:PinHeader_1x01_P2.54mm_Vertical
- added  : Hole 0.6mm ( 2 holes ), Z_mycustom_footprint_lib:Hole 0.6mm ( 2 holes ), F.Cu at (88.5, 119.5)
- added  : Hole 0.6mm ( 2 holes ), Z_mycustom_footprint_lib:Hole 0.6mm ( 2 holes ), F.Cu at (78.1, 108.3)
- added  : Hole 0.6mm ( 2 holes ), Z_mycustom_footprint_lib:Hole 0.6mm ( 2 holes ), F.Cu at (92.0, 119.5)
- added  : Hole 0.6mm ( 2 holes ), Z_mycustom_footprint_lib:Hole 0.6mm ( 2 holes ), F.Cu at (78.1, 104.7)
- added  : Hole 0.6mm ( 2 holes ), Z_mycustom_footprint_lib:Hole 0.6mm ( 2 holes ), F.Cu at (92.0, 122.8)
- added  : Hole 0.6mm ( 2 holes ), Z_mycustom_footprint_lib:Hole 0.6mm ( 2 holes ), F.Cu at (88.5, 122.8)
- added  : Hole 0.6mm ( 2 holes ), Z_mycustom_footprint_lib:Hole 0.6mm ( 2 holes ), F.Cu at (78.1, 106.5)
- added  : Hole 0.6mm ( 2 holes ), Z_mycustom_footprint_lib:Hole 0.6mm ( 2 holes ), F.Cu at (78.1, 101.2)
- added  : Hole 0.6mm ( 2 holes ), Z_mycustom_footprint_lib:Hole 0.6mm ( 2 holes ), F.Cu at (78.1, 110.0)
- added  : Hole 0.6mm ( 2 holes ), Z_mycustom_footprint_lib:Hole 0.6mm ( 2 holes ), F.Cu at (78.1, 103.0)
- added  : Hole 0.6mm ( 2 holes ), Z_mycustom_footprint_lib:Hole 0.6mm ( 2 holes ), F.Cu at (90.2, 122.8)
- added  : Hole 0.6mm ( 2 holes ), Z_mycustom_footprint_lib:Hole 0.6mm ( 2 holes ), F.Cu at (90.2, 119.5)
- added ?: , , F.Cu at (75.0, 100.4)
- added ?: , , F.Cu at (75.0, 104.0)
- added ?: , , F.Cu at (75.0, 107.5)
- added ?: , , F.Cu at (75.0, 108.4)
- added ?: , , F.Cu at (75.0, 103.1)
- added ?: , , F.Cu at (74.9, 109.2)
- added ?: , , F.Cu at (75.0, 106.6)
- added ?: , , F.Cu at (75.0, 101.3)
- added ?: , , F.Cu at (75.0, 104.9)
- added ?: , , F.Cu at (75.0, 105.7)
- added ?: , , F.Cu at (75.0, 102.2)
- added ?: , , F.Cu at (74.9, 110.1)
Routing:
- net /ref3: track 36.6 -> 12.8 mm
- net +3.3VA: track 142.0 -> 121.2 mm
Other:
- outline, holes or cut-outs redrawn

Commit message: y
Parts:
- removed the   at (78.1, 101.2)
- removed the ? at (75.0, 100.4)
- removed the ? at (75.0, 101.3)
- removed kibuzzard-62B56940 (x2): G***, kibuzzard-62B56940
- removed kibuzzard-62B56AED: G***, kibuzzard-62B56AED
- removed kibuzzard-62B56B9A (x2): G***, kibuzzard-62B56B9A
- removed kibuzzard-62B58D0E: G***, kibuzzard-62B58D0E
- added kibuzzard-62B977EB: G***, kibuzzard-62B977EB, F.Cu at (118.4, 101.9)
- added kibuzzard-62B977EB: G***, kibuzzard-62B977EB, F.Cu at (88.1, 131.6)
- added kibuzzard-62B97805: G***, kibuzzard-62B97805, F.Cu at (88.0, 136.3)
- added kibuzzard-62B97805: G***, kibuzzard-62B97805, F.Cu at (118.3, 106.6)
- added kibuzzard-62B97B6B: G***, kibuzzard-62B97B6B, F.Cu at (86.6, 125.5)
- added kibuzzard-62B97B7C: G***, kibuzzard-62B97B7C, F.Cu at (115.1, 58.4)
- moved ? 0.86 mm to (74.8, 101.3)
- moved ? 0.75 mm to (74.8, 102.4)
- moved ? 0.62 mm to (74.8, 103.4)
- moved   0.62 mm to (78.0, 102.4)
- moved ? 0.51 mm to (74.8, 104.4)
- moved   0.50 mm to (78.0, 104.3)
- moved   0.46 mm to (78.0, 106.1)
- moved ? 0.36 mm to (74.8, 106.3)
- moved ? 0.35 mm to (74.8, 105.4)
- moved ? 0.32 mm to (74.8, 107.2)
- moved   0.31 mm to (78.0, 108.0)
- moved ? 0.22 mm to (74.8, 108.2)
- moved ? 0.18 mm to (74.8, 109.1)
- moved   0.16 mm to (78.0, 109.9)
- moved ? 0.13 mm to (74.8, 110.1)
Other:
- outline, holes or cut-outs redrawn

Commit message: f
Parts:
- removed  : Hole 0.6mm ( 2 holes ), Z_mycustom_footprint_lib:Hole 0.6mm ( 2 holes ) (x11)
- removed the ? at (74.8, 102.4)
- removed the ? at (74.8, 108.2)
- removed the ? at (74.8, 109.1)
- removed the ? at (74.8, 106.3)
- removed the ? at (74.8, 104.4)
- removed the ? at (74.8, 105.4)
- removed the ? at (74.8, 101.3)
- removed the ? at (74.8, 110.1)
- removed the ? at (74.8, 103.4)
- removed the ? at (74.8, 107.2)
- removed the H4 at (130.4, 58.3)
- removed the H4 at (130.4, 116.4)
- removed the H4 at (81.5, 116.4)
- added ?: , , F.Cu at (130.4, 58.4)
- added ?: , , F.Cu at (130.5, 116.3)
- added ?: , , F.Cu at (81.4, 116.3)
- added FID5: Fiducial, Z_mycustom_panelization:mouse bites 2.5mm wide 6mm long 0.6mm holes 0.3mm apart streight edges, F.Cu at (75.2, 111.2)
- added FID6: Fiducial, Z_mycustom_panelization:mouse bites 2.5mm wide 6mm long 0.6mm holes 0.3mm apart streight edges, F.Cu at (87.0, 120.0)
- added J9: Conn_01x01, Connector_PinHeader_2.54mm:PinHeader_1x01_P2.54mm_Vertical, F.Cu at (56.5, 100.8)
- moved kibuzzard-62B57119 0.45 mm to (81.1, 107.9)
- renumbered C12 to C10, C10 to C11, C11 to C12, IC2 to IC1, IC1 to IC2, R27 to R10, R10 to R11, R11 to R12, R12 to R13, R13 to R14, R14 to R15, R15 to R16, R16 to R17, R17 to R18, R18 to R19, R19 to R20, R20 to R21, R21 to R22, R22 to R23, R23 to R24, R28 to R25, R24 to R26, R25 to R27, R26 to R28, U8 to U7, U7 to U8
Connections:
- J8 pad 31: unconnected-(J8-Pad31) -> /Comparator2
Routing:
- net /Comparator2: track 4.15 -> 29.9 mm, vias 0 -> 6
- net +3.3VA: track 121.2 -> 124.3 mm
- net /ref3: track 12.8 -> 10.3 mm
- net SS3: track 49.4 -> 50.2 mm
Other:
- outline, holes or cut-outs redrawn
