File: VLC-both/VLC-both.kicad_pcb (KiCad board)
At the start: 2 copper layers, 98.4 x 97.7 mm, 114 parts, among them IC1 TC75S59FU_TE85L,F_, IC2 TC75S59FU_TE85L,F_, J1 dust sense, J2 sound in, J3 40HAT, J4 Conn_01x03, J5 light, J6 proxy, J7 Analof light in, J8 40HAT, J9 Conn_01x01, Q1 Q_NPN_BEC, SW1 SW_SPST, SW2 SW_SPST, U1 LM35-LP, U2 CN240A05, U3 LM4040DBZ-4.1, U4 MCP3008, U5 LM4040DBZ-4.1, U6 MCP3008, U7 LM4040DBZ-3, U8 ADS7041xDCU

Commit message: f
Parts:
- added R29: 0, Resistor_SMD:R_0805_2012Metric, F.Cu at (115.9, 64.4)
Connections:
- J3 pad 3: unconnected-(J3-Pad3) -> /triac_pin
- Q1 pad 2: GND -> Net-(Q1-Pad2)
- R2 pad 1: GND -> Net-(Q1-Pad2)
Routing:
- net /triac_pin: track 0.00 -> 12.0 mm, vias 0 -> 1
- net Net-(Q1-Pad2): track 0.00 -> 4.61 mm
- net GND: track 60.1 -> 56.4 mm, vias 41 -> 40
Other:
- outline, holes or cut-outs redrawn
