File: VLC-both/VLC-both.kicad_sch (KiCad schematic)
At the start: 2 parts, among them J1 40HAT, J3 40HAT

Commit message: h
Parts:
- added C1: 100n, Capacitor_SMD:C_0805_2012Metric, symbol Device:C_Small
- added R1, R2, R3, R4: 10k, Resistor_SMD:R_0805_2012Metric, symbol Device:R_Small
- added U1: MCP3008, Package_SO:SOIC-16_3.9x9.9mm_P1.27mm, symbol Analog_ADC:MCP3008
Connections:
- net +3V3: now also R1.1, R2.1, R3.1, R4.1
- net +5V: now also C1.1, U1.16 (Vdd)
- net GND: now also C1.2, U1.14 (AGND), U1.9 (DGND)
- new net CLK1: R1.2, U1.13 (CLK)
- new net MISO1: R2.2, U1.12 (Dout)
- new net MOSI1: R3.2, U1.11 (Din)
- new net SS1: R4.2, U1.10 (~{CS}/SHDN)

Commit message: Update VLC-both.kicad_sch
Other:
- note added: "Remember to isolate mains. Also references for the ADCs. Screw terminals + pins. Beia logo + cut lines in the middle."
Changed lines of the file:
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@@
     (stroke (width 0) (type default) (color 0 0 0 0))
+  )
+  (text "Remember to isolate mains.\nAlso references for the ADCs.\nScrew terminals + pins.\nBeia logo + cut lines in the middle."
+    (at 157.48 31.115 0)
+    (effects (font (size 1.27 1.27)) (justify left bottom))
   )
   (text "40-Pin HAT Connector" (at 30.48 41.91 0)

Commit message: c
Parts:
- removed U1: MCP3008, Package_SO:SOIC-16_3.9x9.9mm_P1.27mm, symbol Analog_ADC:MCP3008
- added C2: (no value), symbol Device:C_Small
- added C3: 100n-0.1u, Capacitor_SMD:C_0805_2012Metric, symbol Device:C_Small
- added C4, C5, C6, C7: 100n, Capacitor_SMD:C_0805_2012Metric, symbol Device:C_Small
- added J1, J2, J6: (no value), symbol Connector_Generic:Conn_01x03
- added J3: (no value), symbol Connector_Generic:Conn_01x06
- added J4: (no value), symbol Connector_Generic:Conn_01x04
- added Q1: (no value), symbol Device:Q_NPN_BEC
- added R10: 100, Resistor_SMD:R_0805_2012Metric, symbol Device:R_Small
- added R11, R12, R13, R14, R5, R7, R9: 10k, Resistor_SMD:R_0805_2012Metric, symbol Device:R_Small
- added R6, R8: (no value), symbol Device:R_Small
- added TH1: (no value), symbol Device:Thermistor
- added U1: (no value), symbol Sensor_Temperature:LM35-LP
- added U2: (no value), symbol Reference_Voltage:LM4040DBZ-4.1
- added U3, U6: MCP3008, Package_SO:SOIC-16_3.9x9.9mm_P1.27mm, symbol Analog_ADC:MCP3008
- added U4: (no value), symbol Relay_SolidState:S102S01
- added U5: LM4040DBZ-4.1, Package_TO_SOT_SMD:SOT-23, symbol Reference_Voltage:LM4040DBZ-4.1
- C1: value 100n -> (none); footprint Capacitor_SMD:C_0805_2012Metric -> (none)
- R1, R3: value 10k -> (none); footprint Resistor_SMD:R_0805_2012Metric -> (none)
- renumbered J1 to J5, J3 to J7
Connections:
- net +3V3: now also C1.1, J1.2 (Pin_2), J4.3 (Pin_3), R11.1, R12.1, R13.1, R14.1, R5.1, R7.1, R9.1; no longer R1.1, R2.1, R3.1
- net +5V: now also R1.1, R2.1, R3.2, C2.1, C5.1, C7.1, J2.3 (Pin_3), J3.6 (Pin_6), R10.2, U1.1 (+VS), U3.16 (Vdd), U4.3, U6.16 (Vdd); no longer C1.1
- net CLK1: now also J7.23 (BCM11), R11.2, U6.13 (CLK); no longer R1.2
- net GND: now also C2.2, C3.2, C4.2, C5.2, C6.2, C7.2, J1.3 (Pin_3), J2.1 (Pin_1), J3.2 (Pin_2), J3.4 (Pin_4), J4.2 (Pin_2), Q1.2 (E), R8.1, TH1.2, U1.3 (GND), U2.2 (A), U3.14 (AGND), U3.9 (DGND), U5.2 (A), U6.14 (AGND), U6.9 (DGND)
- net MISO1: now also J7.21 (BCM9), R12.2, U6.12 (Dout); no longer R2.2
- net MOSI1: now also J7.19 (BCM10), R13.2, U6.11 (Din); no longer R3.2
- net SS1: now also J7.24 (BCM8), R14.2, U6.10 (~{CS}/SHDN); no longer R4.2
- net MOSI2: now reaches J5.19 (BCM10)
- net MOSI2: now also R7.2, U3.11 (Din)
- net MISO2: now reaches J5.21 (BCM9)
- net MISO2: now also R5.2, U3.12 (Dout)
- net CLK2: now reaches J5.23 (BCM11)
- net CLK2: now also R4.2, U3.13 (CLK)
- net SS2: now reaches J5.24 (BCM8)
- net SS2: now also R9.2, U3.10 (~{CS}/SHDN)
- new net: J3.1 (Pin_1), R1.2
- new net: J6.2 (Pin_2), U4.1
- new net: J6.3 (Pin_3), U4.2
- new net: Q1.1 (B), R6.1, R8.2
- new net: Q1.3 (C), U4.4
- new net ADC0: U1.2 (Vout), U3.1 (CH0), U6.1 (CH0)
- new net ADC1: J4.1 (Pin_1), U3.2 (CH1), U6.2 (CH1)
- new net ADC2: J3.5 (Pin_5), U3.3 (CH2), U6.3 (CH2)
- new net ADC3: C3.1, R2.2, TH1.1, U3.4 (CH3), U6.4 (CH3)
- new net ADC4: U3.5 (CH4), U6.5 (CH4)
- new net ADC5: U3.6 (CH5), U6.6 (CH5)
- new net ADC6: U3.7 (CH6), U6.7 (CH6)
- new net ADC7: U3.8 (CH7), U6.8 (CH7)
- new net V-O: J3.3 (Pin_3)
- new net Vref1: C4.1, C6.1, R10.1, R3.1, U2.1 (K), U3.15 (Vref), U5.1 (K), U6.15 (Vref)
- new net audio_digital_out: J4.4 (Pin_4)
- new net light: J1.1 (Pin_1)
- new net proxy_out: J2.2 (Pin_2)
- new net triac_pin: R6.2
- no-connect marks 0 -> 9
Other:
- note added: "2.7-5.5V BUT 3v3 was used in order to limit TTL to 3v3 max"
- note added: "4.096v ref"
- note added: "HUGE cap for some reason"
- note added: "digital pin 3v3 TTL"
- note added: "digital pin?"
- note added: "~15mA needed"

Commit message: Update VLC-both.kicad_sch
Parts:
- added IC?: (no value), symbol SamacSys_Parts:TC75S59FU_TE85L,F_
- C1: value (none) -> 100n-0.1u; footprint (none) -> Capacitor_SMD:C_0805_2012Metric
- C2: value (none) -> 220u; footprint (none) -> Capacitor_SMD:C_0805_2012Metric
- J1: value (none) -> light; footprint (none) -> Connector_PinHeader_2.54mm:PinHeader_1x03_P2.54mm_Vertical
- J2: value (none) -> proxy; footprint (none) -> Connector_PinHeader_2.54mm:PinHeader_1x03_P2.54mm_Vertical
- J3: value (none) -> dust sense; footprint (none) -> Connector_PinHeader_2.54mm:PinHeader_1x06_P2.54mm_Vertical
- J4: value (none) -> sound in; footprint (none) -> Connector_PinHeader_2.54mm:PinHeader_1x04_P2.54mm_Vertical
- J6: value (none) -> Conn_01x03; footprint (none) -> TerminalBlock:TerminalBlock_Altech_AK300-3_P5.00mm
- Q1: value (none) -> Q_NPN_BEC; footprint (none) -> Package_TO_SOT_SMD:SOT-23
- R1: value (none) -> 150; footprint (none) -> Resistor_SMD:R_0805_2012Metric
- R3: value (none) -> 100; footprint (none) -> Resistor_SMD:R_0805_2012Metric
- R6: value (none) -> 90k; footprint (none) -> Resistor_SMD:R_0805_2012Metric
- R8: value (none) -> DNP; footprint (none) -> Resistor_SMD:R_0805_2012Metric
- TH1: value (none) -> Thermistor
- U1: value (none) -> LM35-LP; footprint (none) -> Connector_PinHeader_2.54mm:PinHeader_1x03_P2.54mm_Vertical
- U2: value (none) -> LM4040DBZ-4.1; footprint (none) -> Package_TO_SOT_SMD:SOT-23
- U4: value (none) -> CN240A05; footprint (none) -> Package_SIP:SIP4_Sharp-SSR_P7.62mm_Straight
Changed lines of the file:
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@@
       (effects (font (size 1.27 1.27)) (justify left))
     )
-    (property "Value" "" (id 1) (at 38.1 189.23 0)
-      (effects (font (size 1.27 1.27)) (justify left))
-    )
-    (property "Footprint" "" (id 2) (at 39.37 187.96 0)
+    (property "Value" "150" (id 1) (at 38.1 189.23 0)
+      (effects (font (size 1.27 1.27)) (justify left))
+    )
+    (property "Footprint" "Resistor_SMD:R_0805_2012Metric" (id 2) (at 39.37 187.96 0)
       (effects (font (size 1.27 1.27)) hide)
     )
@@
       (effects (font (size 1.27 1.27)) (justify left))
     )
-    (property "Value" "" (id 1) (at 222.25 167.0049 0)
-      (effects (font (size 1.27 1.27)) (justify left))
-    )
-    (property "Footprint" "" (id 2) (at 219.075 165.735 0)
+    (property "Value" "Conn_01x03" (id 1) (at 222.25 167.0049 0)
+      (effects (font (size 1.27 1.27)) (justify left))
+    )
+    (property "Footprint" "TerminalBlock:TerminalBlock_Altech_AK300-3_P5.00mm" (id 2) (at 219.075 165.735 0)
       (effects (font (size 1.27 1.27)) hide)
     )
@@
       (effects (font (size 1.27 1.27)) (justify left))
     )
-    (property "Value" "" (id 1) (at 93.98 268.6049 0)
+    (property "Value" "Thermistor" (id 1) (at 93.98 268.6049 0)
       (effects (font (size 1.27 1.27)) (justify left))
     )
@@
       (effects (font (size 1.27 1.27)) (justify left))
     )
-    (property "Value" "" (id 1) (at 167.005 186.055 0)
-      (effects (font (size 1.27 1.27)) (justify left))
-    )
-    (property "Footprint" "" (id 2) (at 168.275 184.785 0)
+    (property "Value" "90k" (id 1) (at 167.005 186.055 0)
+      (effects (font (size 1.27 1.27)) (justify left))
+    )
+    (property "Footprint" "Resistor_SMD:R_0805_2012Metric" (id 2) (at 168.275 184.785 0)
       (effects (font (size 1.27 1.27)) hide)
     )
@@
     (in_bom yes) (on_board yes)
     (property "Reference" "J2" (id 0) (at 28.575 207.01 0))
-    (property "Value" "" (id 1) (at 28.575 209.55 0))
-    (property "Footprint" "" (id 2) (at 28.575 216.535 0)
+    (property "Value" "proxy" (id 1) (at 28.575 209.55 0))
+    (property "Footprint" "Connector_PinHeader_2.54mm:PinHeader_1x03_P2.54mm_Vertical" (id 2) (at 28.575 216.535 0)
       (effects (font (size 1.27 1.27)) hide)
     )
@@
       (effects (font (size 1.27 1.27)) (justify left))
     )
-    (property "Value" "" (id 1) (at 102.235 60.96 90)
-      (effects (font (size 1.27 1.27)) (justify left))
-    )
-    (property "Footprint" "" (id 2) (at 115.57 60.325 0)
+    (property "Value" "LM4040DBZ-4.1" (id 1) (at 102.235 60.96 90)
+      (effects (font (size 1.27 1.27)) (justify left))
+    )
+    (property "Footprint" "Package_TO_SOT_SMD:SOT-23" (id 2) (at 115.57 60.325 0)
       (effects (font (size 1.27 1.27) italic) hide)
     )
@@
     (in_bom yes) (on_board yes)
     (property "Reference" "J4" (id 0) (at 30.48 140.97 0))
-    (property "Value" "" (id 1) (at 30.48 143.51 0))
-    (property "Footprint" "" (id 2) (at 30.48 153.035 0)
+    (property "Value" "sound in" (id 1) (at 30.48 143.51 0))
+    (property "Footprint" "Connector_PinHeader_2.54mm:PinHeader_1x04_P2.54mm_Vertical" (id 2) (at 30.48 153.035 0)
       (effects (font (size 1.27 1.27)) hide)
     )
@@
       (effects (font (size 1.27 1.27)) (justify left))
     )
-    (property "Value" "" (id 1) (at 119.38 49.53 0)
-      (effects (font (size 1.27 1.27)) (justify left))
-    )
-    (property "Footprint" "" (id 2) (at 120.65 50.8 0)
+    (property "Value" "100" (id 1) (at 119.38 49.53 0)
+      (effects (font (size 1.27 1.27)) (justify left))
+    )
+    (property "Footprint" "Resistor_SMD:R_0805_2012Metric" (id 2) (at 120.65 50.8 0)
       (effects (font (size 1.27 1.27)) hide)
     )
@@
       (effects (font (size 1.27 1.27)) (justify left))
     )
-    (property "Value" "" (id 1) (at 187.96 186.0549 0)
-      (effects (font (size 1.27 1.27)) (justify left))
-    )
-    (property "Footprint" "" (id 2) (at 187.325 182.245 0)
+    (property "Value" "Q_NPN_BEC" (id 1) (at 187.96 186.0549 0)
+      (effects (font (size 1.27 1.27)) (justify left))
+    )
+    (property "Footprint" "Package_TO_SOT_SMD:SOT-23" (id 2) (at 187.325 182.245 0)
       (effects (font (size 1.27 1.27)) hide)
     )
@@
       (effects (font (size 1.27 1.27)) (justify right))
     )
-    (property "Value" "" (id 1) (at 21.59 125.7299 0)
+    (property "Value" "LM35-LP" (id 1) (at 21.59 125.7299 0)
       (effects (font (size 1.27 1.27)) (justify right))
     )
-    (property "Footprint" "" (id 2) (at 31.75 130.81 0)
+    (property "Footprint" "Connector_PinHeader_2.54mm:PinHeader_1x03_P2.54mm_Vertical" (id 2) (at 31.75 130.81 0)
       (effects (font (size 1.27 1.27)) (justify left) hide)
     )
@@
     (in_bom yes) (on_board yes)
     (property "Reference" "J1" (id 0) (at 27.94 227.965 0))
-    (property "Value" "" (id 1) (at 27.94 230.505 0))
-    (property "Footprint" "" (id 2) (at 27.94 237.49 0)
+    (property "Value" "light" (id 1) (at 27.94 230.505 0))
+    (property "Footprint" "Connector_PinHeader_2.54mm:PinHeader_1x03_P2.54mm_Vertical" (id 2) (at 27.94 237.49 0)
       (effects (font (size 1.27 1.27)) hide)
     )
@@
       (effects (font (size 1.27 1.27)) (justify left))
     )
-    (property "Value" "" (id 1) (at 46.355 194.3162 0)
-      (effects (font (size 1.27 1.27)) (justify left))
-    )
-    (property "Footprint" "" (id 2) (at 43.815 193.04 0)
+    (property "Value" "220u" (id 1) (at 46.355 194.3162 0)
+      (effects (font (size 1.27 1.27)) (justify left))
+    )
+    (property "Footprint" "Capacitor_SMD:C_0805_2012Metric" (id 2) (at 43.815 193.04 0)
       (effects (font (size 1.27 1.27)) hide)
     )
@@
       (effects (font (size 1.27 1.27)) (justify left))
     )
-    (property "Value" "" (id 1) (at 43.815 243.2112 0)
-      (effects (font (size 1.27 1.27)) (justify left))
-    )
-    (property "Footprint" "" (id 2) (at 41.275 241.935 0)
+    (property "Value" "100n-0.1u" (id 1) (at 43.815 243.2112 0)
+      (effects (font (size 1.27 1.27)) (justify left))
+    )
+    (property "Footprint" "Capacitor_SMD:C_0805_2012Metric" (id 2) (at 41.275 241.935 0)
       (effects (font (size 1.27 1.27)) hide)
     )
@@
       (effects (font (size 1.27 1.27)) (justify left))
     )
-    (property "Value" "" (id 1) (at 180.34 188.595 0)
-      (effects (font (size 1.27 1.27)) (justify left))
-    )
-    (property "Footprint" "" (id 2) (at 174.625 189.865 0)
+    (property "Value" "DNP" (id 1) (at 180.34 188.595 0)
+      (effects (font (size 1.27 1.27)) (justify left))
+    )
+    (property "Footprint" "Resistor_SMD:R_0805_2012Metric" (id 2) (at 174.625 189.865 0)
       (effects (font (size 1.27 1.27)) hide)
     )
@@
     (pin "1")
   )
+  (symbol (lib_id "SamacSys_Parts:TC75S59FU_TE85L,F_") (at 308.61 201.93 0) (unit 1)
+    (in_bom yes) (on_board yes) (fields_autoplaced)
+    (property "Reference" "IC?" (id 0) (at 325.12 194.31 0))
+    (property "Value" "" (id 1) (at 325.12 196.85 0))
+    (property "Footprint" "" (id 2) (at 337.82 199.39 0)
+      (effects (font (size 1.27 1.27)) (justify left) hide)
+    )
+    (property "Datasheet" "https://componentsearchengine.com/Datasheets/1/TC75S59FU(TE85L,F).pdf" (id 3) (at 337.82 201.93 0)
+      (effects (font (size 1.27 1.27)) (justify left) hide)
+    )
+    (property "Description" "OpAmp,Comparator,C-MOS" (id 4) (at 337.82 204.47 0)
+      (effects (font (size 1.27 1.27)) (justify left) hide)
+    )
+    (property "Height" "1.1" (id 5) (at 337.82 207.01 0)
+      (effects (font (size 1.27 1.27)) (justify left) hide)
+    )
+    (property "Mouser Part Number" "757-TC75S59FUTE85LF" (id 6) (at 337.82 209.55 0)
+      (effects (font (size 1.27 1.27)) (justify left) hide)
+    )
+    (property "Mouser Price/Stock" "https://www.mouser.com/Search/Refine.aspx?Keyword=757-TC75S59FUTE85LF" (id 7) (at 337.82 212.09 0)
+      (effects (font (size 1.27 1.27)) (justify left) hide)
+    )
+    (property "Manufacturer_Name" "Toshiba" (id 8) (at 337.82 214.63 0)
+      (effects (font (size 1.27 1.27)) (justify left) hide)
+    )
+    (property "Manufacturer_Part_Number" "TC75S59FU(TE85L,F)" (id 9) (at 337.82 217.17 0)
+      (effects (font (size 1.27 1.27)) (justify left) hide)
+    )
+    (pin "1")
+    (pin "2")
+    (pin "3")
+    (pin "4")
+    (pin "5")
+  )
   (symbol (lib_id "Connector_Generic:Conn_01x06") (at 29.21 182.88 180) (unit 1)
     (in_bom yes) (on_board yes)
     (property "Reference" "J3" (id 0) (at 29.21 168.91 0))
-    (property "Value" "" (id 1) (at 29.21 171.45 0))
-    (property "Footprint" "" (id 2) (at 29.21 182.88 0)
+    (property "Value" "dust sense" (id 1) (at 29.21 171.45 0))
+    (property "Footprint" "Connector_PinHeader_2.54mm:PinHeader_1x06_P2.54mm_Vertical" (id 2) (at 29.21 182.88 0)
       (effects (font (size 1.27 1.27)) hide)
     )
@@
     (in_bom yes) (on_board yes) (fields_autoplaced)
     (property "Reference" "U4" (id 0) (at 194.31 158.75 0))
-    (property "Value" "" (id 1) (at 194.31 161.29 0))
-    (property "Footprint" "" (id 2) (at 189.23 173.355 0)
+    (property "Value" "CN240A05" (id 1) (at 194.31 161.29 0))
+    (property "Footprint" "Package_SIP:SIP4_Sharp-SSR_P7.62mm_Straight" (id 2) (at 189.23 173.355 0)
       (effects (font (size 1.27 1.27) italic) (justify left) hide)
     )
@@
       (reference "C7") (unit 1) (value "100n") (footprint "Capacitor_SMD:C_0805_2012Metric")
     )
+    (path "/e416fb41-ee88-462f-847d-7d5eaeae8cc4"
+      (reference "IC?") (unit 1) (value "TC75S59FU_TE85L,F_") (footprint "TC75S59FUTE85LF")
+    )
     (path "/9426f8fe-a299-4cfd-bc9c-030ea7569cf6"

Commit message: r
Parts:
- added C8, C9: 100n, Capacitor_SMD:C_0805_2012Metric, symbol Device:C_Small
- added IC1: TC75S59FU_TE85L,F_, TC75S59FUTE85LF, symbol SamacSys_Parts:TC75S59FU_TE85L,F_
- added J8: sound in, Connector_PinHeader_2.54mm:PinHeader_1x04_P2.54mm_Vertical, symbol Connector_Generic:Conn_01x04
- added R15, R16: DNP, Resistor_SMD:R_0805_2012Metric, symbol Device:R_Small
- added R17, R19: 10k, Resistor_SMD:R_0805_2012Metric, symbol Device:R_Small
- added R18: 20k, Resistor_SMD:R_0805_2012Metric, symbol Device:R_Small
- added RV1, RV2: R_Potentiometer, Potentiometer_THT:Potentiometer_Piher_PT-6-V_Vertical, symbol Device:R_Potentiometer
- IC2: renamed from IC?; value (none) -> TC75S59FU_TE85L,F_; footprint (none) -> TC75S59FUTE85LF
- TH1: footprint (none) -> Connector_PinHeader_2.54mm:PinHeader_1x02_P2.54mm_Vertical
Connections:
- net +3V3: now also IC2.5 (VDD), C8.2, C9.2, IC1.5 (VDD)
- net +5V: no longer C2.1
- net ADC0: now also J8.4 (Pin_4)
- net ADC1: no longer U6.2 (CH1)
- net ADC2: no longer U6.3 (CH2)
- net ADC3: no longer U6.4 (CH3)
- net ADC4: no longer U6.5 (CH4)
- net ADC5: no longer U6.6 (CH5)
- net ADC6: no longer U6.7 (CH6)
- net ADC7: no longer U6.8 (CH7)
- net GND: now also IC2.2 (VSS), C8.1, C9.1, IC1.2 (VSS), J8.1 (Pin_1), R19.1, RV1.3, RV2.3
- net V-O: now also J5.40 (BCM21)
- net Vref1: now also R15.1, R17.2, RV1.1
- net audio_digital_out: now also J5.38 (BCM20)
- net proxy_out: now also J5.36 (BCM16)
- net Comparator1: now reaches J7.38 (BCM20)
- net Comparator1: now also IC2.4 (OUT)
- net Comparator2: now reaches J7.40 (BCM21)
- net Comparator2: now also IC1.4 (OUT)
- net at J3.1 (Pin_1), R1.2: now also C2.1
- net at IC2.1 (IN_(-)): now also RV2.2
- net at IC2.3 (IN_(+)): now also RV1.2
- new net: IC1.3 (IN_(+)), R16.2, R18.1, R19.2
- new net: R17.1, R18.2
- new net: R15.2, R16.1
- new net IN1: IC1.1 (IN_(-)), J8.3 (Pin_3)
- new net IN2: J8.2 (Pin_2), RV2.1
- no-connect marks 9 -> 56
Other:
- moved on the sheet: R1

Commit message: t
Parts:
- removed J8: sound in, Connector_PinHeader_2.54mm:PinHeader_1x04_P2.54mm_Vertical, symbol Connector_Generic:Conn_01x04
- added J7: (no value), symbol Connector_Generic:Conn_01x06
- added R15, R16: (no value), symbol Device:R_Small
- added U7: (no value), symbol Analog_ADC:ADS7041xDCU
- C1: renamed from C2; value 220u -> (none); footprint Capacitor_SMD:C_0805_2012Metric -> (none)
- IC1, IC2: footprint TC75S59FUTE85LF -> (none)
- renumbered C3 to C2, C4 to C3, C5 to C4, C1 to C5, C8 to C7, C9 to C8, C7 to C9, J3 to J1, J4 to J2, J5 to J3, J6 to J4, J1 to J5, J2 to J6, J7 to J8, R6 to R1, R15 to R10, R16 to R11, R17 to R12, R18 to R13, R19 to R14, R10 to R17, R11 to R18, R12 to R19, R8 to R2, R13 to R20, R14 to R21, R1 to R3, R3 to R4, R2 to R5, R4 to R6, R5 to R7, R7 to R8, U4 to U2, U2 to U3, U3 to U4
Connections:
- net ADC0: no longer U6.1 (CH0)
- net Comparator2: now also R16.2
- net GND: now also J7.1 (Pin_1), U7.5 (AINM), U7.8 (GND)
- net IN1: now also J7.4 (Pin_4), R15.1; no longer IC1.1 (IN_(-))
- net IN2: now also RV1.1, J7.2 (Pin_2); no longer RV2.1
- net Vref1: now also RV2.1; no longer C3.1, R4.1, RV1.1, U3.1 (K), U4.15 (Vref)
- net at R11.2, R13.1, R14.2: now also IC1.1 (IN_(-)); no longer IC1.3 (IN_(+))
- net L2: now reaches J4.1 (Pin_1)
- net L2: now also U2.2
- net L1: now reaches J4.2 (Pin_2), U2.1
- net at J4.3 (Pin_3): no longer U2.2
- new net: IC1.3 (IN_(+)), R15.2, R16.1
- new net ADC0_1: J7.3 (Pin_3), U6.1 (CH0)
- new net ADC1_1: J7.5 (Pin_5), U7.6 (AINP)
- new net Vref2: C3.1, R4.1, U3.1 (K), U4.15 (Vref)
Other:
- moved on the sheet: C1, C2, C5, C6, C7, C8, C9, IC1, IC2, J1, J2, J4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
