File: VLC-both/VLC-both.kicad_sch (KiCad schematic)
At the start: 51 parts, among them IC1 TC75S59FU_TE85L,F_, IC2 TC75S59FU_TE85L,F_, J1 dust sense, J2 sound in, J3 40HAT, J4 Conn_01x03, J5 light, J6 proxy, J7 Analof light in, J8 40HAT, Q1 Q_NPN_BEC, U1 LM35-LP, U2 CN240A05, U3 LM4040DBZ-4.1, U4 MCP3008, U5 LM4040DBZ-4.1, U6 MCP3008, U7 ADS7041xDCU

Commit message: r
Parts:
- added C10, C11, C12: 1u, Capacitor_SMD:C_0805_2012Metric, symbol Device:C_Small
- added FID1, FID3: Fiducial, Fiducial:Fiducial_0.5mm_Mask1mm, symbol Mechanical:Fiducial
- added FID2, FID4: Fiducial, Symbol:WEEE-Logo_4.2x6mm_SilkScreen, symbol Mechanical:Fiducial
- added R22: DNP, Resistor_SMD:R_0805_2012Metric, symbol Device:R_Small
- added R23: 100, Resistor_SMD:R_0805_2012Metric, symbol Device:R_Small
- added R24, R25, R26: 10k, Resistor_SMD:R_0805_2012Metric, symbol Device:R_Small
- added U8: LM4040DBZ-3, Package_TO_SOT_SMD:SOT-23, symbol Reference_Voltage:LM4040DBZ-3
Connections:
- net +3.3VA: now also U7.1 (DVDD), C11.1, R23.2, R24.1, R25.1, R26.1
- net ADC1_1: now also R22.2; no longer U7.6 (AINP)
- net Comparator1: now also J8.37 (BCM26); no longer J8.38 (BCM20)
- net Comparator2: no longer J8.40 (BCM21)
- net GND: now also C10.1, C11.2, C12.2, U8.2 (A)
- net V-O: now also J3.35 (BCM19); no longer J3.40 (BCM21)
- net audio_digital_out: now also J3.15 (BCM22); no longer J3.38 (BCM20)
- net light: now also J3.40 (BCM21)
- net proxy_out: now also J3.37 (BCM26); no longer J3.36 (BCM16)
- net MISO3: now reaches J8.35 (BCM19)
- net MISO3: now also U7.3 (SDO), R26.2
- net SS3: now reaches J8.36 (BCM16)
- net SS3: now also U7.4 (~{CS}), R24.2
- net IN-2: now reaches IC1.1 (IN_(-)), R11.2, R13.1, R14.2
- net IN+2: now reaches IC1.3 (IN_(+)), R15.2, R16.1
- net IN-1: now reaches IC2.1 (IN_(-)), RV2.2
- net CLK3: now reaches U7.2 (SCLK)
- net CLK3: now also J8.40 (BCM21), R25.2
- net ref3: now reaches U7.7 (AVDD)
- net ref3: now also C10.2, R23.1, U8.1 (K)
- net IN+1: now reaches IC2.3 (IN_(+)), RV1.2
- new net input: C12.1, R22.1, U7.6 (AINP)
- no-connect marks 58 -> 57
Other:
- note added: "GRAFICA"

Commit message: r
Parts:
- renumbered IC2 to IC1, IC1 to IC2
Changed lines of the file:
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@@
   (symbol (lib_id "SamacSys_Parts:TC75S59FU_TE85L,F_") (at 235.585 189.865 0) (unit 1)
     (in_bom yes) (on_board yes) (fields_autoplaced)
-    (property "Reference" "IC1" (id 0) (at 252.095 182.245 0))
-    (property "Value" "TC75S59FU_TE85L,F_" (id 1) (at 252.095 184.785 0))
+    (property "Reference" "IC2" (id 0) (at 252.095 181.61 0))
+    (property "Value" "TC75S59FU_TE85L,F_" (id 1) (at 252.095 184.15 0))
     (property "Footprint" "SamacSys_Parts:TC75S59FUTE85LF" (id 2) (at 264.795 187.325 0)
       (effects (font (size 1.27 1.27)) (justify left) hide)
@@
   (symbol (lib_id "SamacSys_Parts:TC75S59FU_TE85L,F_") (at 241.3 241.3 0) (unit 1)
     (in_bom yes) (on_board yes) (fields_autoplaced)
-    (property "Reference" "IC2" (id 0) (at 257.81 233.68 0))
+    (property "Reference" "IC1" (id 0) (at 257.81 233.68 0))
     (property "Value" "TC75S59FU_TE85L,F_" (id 1) (at 257.81 236.22 0))
     (property "Footprint" "SamacSys_Parts:TC75S59FUTE85LF" (id 2) (at 270.51 238.76 0)
@@
       (reference "FID4") (unit 1) (value "Fiducial") (footprint "Symbol:WEEE-Logo_4.2x6mm_SilkScreen")
     )
+    (path "/e416fb41-ee88-462f-847d-7d5eaeae8cc4"
+      (reference "IC1") (unit 1) (value "TC75S59FU_TE85L,F_") (footprint "SamacSys_Parts:TC75S59FUTE85LF")
+    )
     (path "/c11b21cf-cc07-4f01-9758-f871f431a3c0"
-      (reference "IC1") (unit 1) (value "TC75S59FU_TE85L,F_") (footprint "SamacSys_Parts:TC75S59FUTE85LF")
-    )
-    (path "/e416fb41-ee88-462f-847d-7d5eaeae8cc4"
       (reference "IC2") (unit 1) (value "TC75S59FU_TE85L,F_") (footprint "SamacSys_Parts:TC75S59FUTE85LF")
     )

Commit message: f
Parts:
- added J9: (no value), symbol Connector_Generic:Conn_01x01
- added R27, R28: 10k, Resistor_SMD:R_0805_2012Metric, symbol Device:R_Small
- added SW1: SW_SPST, SamacSys_Parts:PTS526SM15SMTR2LFS, symbol Switch:SW_SPST
- added SW2: (no value), symbol Switch:SW_SPST
Connections:
- net +3.3VA: now also J9.1 (Pin_1), R28.2
- net +3V3: now also R27.2
- net GND: now also SW1.1 (A), SW2.1 (A)
- net reset2: now reaches J8.11 (BCM17)
- net reset2: now also R28.1, SW2.2 (B)
- net reset1: now reaches J3.11 (BCM17)
- net reset1: now also R27.1, SW1.2 (B)

Commit message: f
Parts:
- added FID5, FID6: Fiducial, Z_mycustom_panelization:mouse bites 2.5mm wide 6mm long 0.6mm holes 0.3mm apart streight edges, symbol Mechanical:Fiducial
- J9: value (none) -> Conn_01x01; footprint (none) -> Connector_PinHeader_2.54mm:PinHeader_1x01_P2.54mm_Vertical
- SW2: value (none) -> SW_SPST; footprint (none) -> SamacSys_Parts:PTS526SM15SMTR2LFS
- renumbered C12 to C10, C10 to C11, C11 to C12, IC2 to IC1, IC1 to IC2, R27 to R10, R10 to R11, R11 to R12, R12 to R13, R13 to R14, R14 to R15, R15 to R16, R16 to R17, R17 to R18, R18 to R19, R19 to R20, R20 to R21, R21 to R22, R22 to R23, R23 to R24, R28 to R25, R24 to R26, R25 to R27, R26 to R28, U8 to U7, U7 to U8
Connections:
- net Comparator2: now also J8.31 (BCM6)
Other:
- note added: "panelization"

Commit message: f
Parts:
- added R29: 0, Resistor_SMD:R_0805_2012Metric, symbol Device:R_Small
Connections:
- net GND: now also R29.1; no longer Q1.2 (E), R2.1
- net triac_pin: now also J3.3 (BCM2)
- new net: Q1.2 (E), R2.1, R29.2
Other:
- moved on the sheet: J4, Q1, R1, R2, U2
