File: VLC-both/_autosave-VLC-both.kicad_pcb (KiCad board)
At the start: 2 copper layers, 98.4 x 97.7 mm, 58 parts, among them IC1 TC75S59FU_TE85L,F_, IC2 TC75S59FU_TE85L,F_, J1 dust sense, J2 sound in, J3 40HAT, J4 Conn_01x03, J5 light, J6 proxy, J7 Analof light in, J8 40HAT, Q1 Q_NPN_BEC, U1 LM35-LP, U2 CN240A05, U3 LM4040DBZ-4.1, U4 MCP3008, U5 LM4040DBZ-4.1, U6 MCP3008, U7 ADS7041xDCU

Commit message: f
Parts:
- moved C5 0.10 mm to (119.8, 113.7)
Connections:
- C7 pad 2: +3V3 -> +3.3VA
- C8 pad 2: +3V3 -> +3.3VA
- C9 pad 1: +5V -> +5VA
- IC1 pad 5: +3V3 -> +3.3VA
- IC2 pad 5: +3V3 -> +3.3VA
- J3 pad 15: unconnected-(J3-Pad15) -> /audio_digital_out
- J3 pad 35: unconnected-(J3-Pad35) -> /V-O
- J3 pad 36: /proxy_out -> unconnected-(J3-Pad36)
- J3 pad 37: unconnected-(J3-Pad37) -> /proxy_out
- J3 pad 38: /audio_digital_out -> unconnected-(J3-Pad38)
- J3 pad 40: /V-O -> unconnected-(J3-Pad40)
- J8 pad 1: +3V3 -> +3.3VA
- J8 pad 17: +3V3 -> +3.3VA
- J8 pad 2: +5V -> +5VA
- J8 pad 4: +5V -> +5VA
- R17 pad 2: +5V -> +5VA
- R18 pad 1: +3V3 -> +3.3VA
- R19 pad 1: +3V3 -> +3.3VA
- R20 pad 1: +3V3 -> +3.3VA
- R21 pad 1: +3V3 -> +3.3VA
- U6 pad 16: +5V -> +5VA
Routing:
- net /audio_digital_out: track 0.00 -> 50.0 mm, vias 0 -> 5
- net +3V3: track 71.3 -> 116.4 mm, vias 5 -> 9
- net /proxy_out: track 0.00 -> 27.7 mm
- net /V-O: track 51.2 -> 57.2 mm
- net +5V: track 142.7 -> 145.2 mm
- added copper zone on F.Cu, net +5V
- added copper zone on F.Cu, net +5VA
