File: VLC-both/_autosave-VLC-both.kicad_sch (KiCad schematic)
At the start: 51 parts, among them IC1 TC75S59FU_TE85L,F_, IC2 TC75S59FU_TE85L,F_, J1 dust sense, J2 sound in, J3 40HAT, J4 Conn_01x03, J5 light, J6 proxy, J7 Analof light in, J8 40HAT, Q1 Q_NPN_BEC, U1 LM35-LP, U2 CN240A05, U3 LM4040DBZ-4.1, U4 MCP3008, U5 LM4040DBZ-4.1, U6 MCP3008, U7 ADS7041xDCU

Commit message: f
Connections:
- net V-O: now also J3.35 (BCM19); no longer J3.40 (BCM21)
- net audio_digital_out: now also J3.15 (BCM22); no longer J3.38 (BCM20)
- net proxy_out: now also J3.37 (BCM26); no longer J3.36 (BCM16)
Changed lines of the file:
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@@
     (effects (font (size 1.27 1.27)) (justify right bottom))
   )
-  (label "proxy_out" (at 76.2 91.44 0)
-    (effects (font (size 1.27 1.27)) (justify left bottom))
+  (label "proxy_out" (at 33.02 93.98 180)
+    (effects (font (size 1.27 1.27)) (justify right bottom))
   )
   (label "light" (at 139.065 217.17 0)
@@
     (effects (font (size 1.27 1.27)) (justify right bottom))
   )
-  (label "audio_digital_out" (at 74.93 93.98 0)
-    (effects (font (size 1.27 1.27)) (justify left bottom))
+  (label "audio_digital_out" (at 31.75 66.04 180)
+    (effects (font (size 1.27 1.27)) (justify right bottom))
   )
   (label "ADC4" (at 116.84 81.915 180)
@@
     (effects (font (size 1.27 1.27)) (justify right bottom))
   )
-  (label "V-O" (at 74.93 96.52 0)
+  (label "V-O" (at 34.29 91.44 0)
     (effects (font (size 1.27 1.27)) (justify left bottom))
   )
@@
   (symbol (lib_id "power:+3.3VA") (at 219.075 54.61 90) (unit 1)
     (in_bom yes) (on_board yes)
-    (property "Reference" "#PWR?" (id 0) (at 222.885 54.61 0)
+    (property "Reference" "#PWR0107" (id 0) (at 222.885 54.61 0)
       (effects (font (size 1.27 1.27)) hide)
     )
@@
   (symbol (lib_id "power:+3.3VA") (at 285.115 189.865 0) (unit 1)
     (in_bom yes) (on_board yes) (fields_autoplaced)
-    (property "Reference" "#PWR?" (id 0) (at 285.115 193.675 0)
+    (property "Reference" "#PWR0101" (id 0) (at 285.115 193.675 0)
       (effects (font (size 1.27 1.27)) hide)
     )
@@
   (symbol (lib_id "power:+3.3VA") (at 219.71 34.29 0) (unit 1)
     (in_bom yes) (on_board yes) (fields_autoplaced)
-    (property "Reference" "#PWR?" (id 0) (at 219.71 38.1 0)
+    (property "Reference" "#PWR0106" (id 0) (at 219.71 38.1 0)
       (effects (font (size 1.27 1.27)) hide)
     )
@@
   (symbol (lib_id "power:+5VA") (at 281.305 98.425 0) (unit 1)
     (in_bom yes) (on_board yes) (fields_autoplaced)
-    (property "Reference" "#PWR?" (id 0) (at 281.305 102.235 0)
+    (property "Reference" "#PWR0102" (id 0) (at 281.305 102.235 0)
       (effects (font (size 1.27 1.27)) hide)
     )
@@
   (symbol (lib_id "power:+3.3VA") (at 290.83 241.3 0) (unit 1)
     (in_bom yes) (on_board yes) (fields_autoplaced)
-    (property "Reference" "#PWR?" (id 0) (at 290.83 245.11 0)
+    (property "Reference" "#PWR0105" (id 0) (at 290.83 245.11 0)
       (effects (font (size 1.27 1.27)) hide)
     )
@@
   (symbol (lib_id "power:+5VA") (at 272.415 34.29 0) (unit 1)
     (in_bom yes) (on_board yes) (fields_autoplaced)
-    (property "Reference" "#PWR?" (id 0) (at 272.415 38.1 0)
+    (property "Reference" "#PWR0104" (id 0) (at 272.415 38.1 0)
       (effects (font (size 1.27 1.27)) hide)
     )
@@
   (symbol (lib_id "power:+3.3VA") (at 309.245 113.03 0) (unit 1)
     (in_bom yes) (on_board yes) (fields_autoplaced)
-    (property "Reference" "#PWR?" (id 0) (at 309.245 116.84 0)
+    (property "Reference" "#PWR0103" (id 0) (at 309.245 116.84 0)
       (effects (font (size 1.27 1.27)) hide)
     )
@@
       (reference "#PWR063") (unit 1) (value "GND") (footprint "")
     )
+    (path "/3da04cc1-8be9-47b2-96a8-cfa93a0bc2b0"
+      (reference "#PWR0101") (unit 1) (value "+3.3VA") (footprint "")
+    )
+    (path "/57ddad74-9948-40fd-9d81-7c857179087b"
+      (reference "#PWR0102") (unit 1) (value "+5VA") (footprint "")
+    )
+    (path "/ff5abd15-ec5d-4dcc-935f-4e4184386954"
+      (reference "#PWR0103") (unit 1) (value "+3.3VA") (footprint "")
+    )
+    (path "/f9290c0e-0ff4-40eb-9f98-514f56d6765b"
+      (reference "#PWR0104") (unit 1) (value "+5VA") (footprint "")
+    )
+    (path "/7a67054d-a23f-4347-9965-a8c2eb887fc2"
+      (reference "#PWR0105") (unit 1) (value "+3.3VA") (footprint "")
+    )
+    (path "/452cb936-74e0-4ed3-a548-aa9f5c0554cf"
+      (reference "#PWR0106") (unit 1) (value "+3.3VA") (footprint "")
+    )
     (path "/00f2c8f5-cdc0-4ca3-aee6-313126ba6106"
-      (reference "#PWR?") (unit 1) (value "+3.3VA") (footprint "")
-    )
-    (path "/3da04cc1-8be9-47b2-96a8-cfa93a0bc2b0"
-      (reference "#PWR?") (unit 1) (value "+3.3VA") (footprint "")
-    )
-    (path "/452cb936-74e0-4ed3-a548-aa9f5c0554cf"
-      (reference "#PWR?") (unit 1) (value "+3.3VA") (footprint "")
-    )
-    (path "/57ddad74-9948-40fd-9d81-7c857179087b"
-      (reference "#PWR?") (unit 1) (value "+5VA") (footprint "")
-    )
-    (path "/7a67054d-a23f-4347-9965-a8c2eb887fc2"
-      (reference "#PWR?") (unit 1) (value "+3.3VA") (footprint "")
-    )
-    (path "/f9290c0e-0ff4-40eb-9f98-514f56d6765b"
-      (reference "#PWR?") (unit 1) (value "+5VA") (footprint "")
-    )
-    (path "/ff5abd15-ec5d-4dcc-935f-4e4184386954"
-      (reference "#PWR?") (unit 1) (value "+3.3VA") (footprint "")
+      (reference "#PWR0107") (unit 1) (value "+3.3VA") (footprint "")
     )
     (path "/9c69993a-a8b6-4904-a7cf-8e8126089be0"
